File: hw-smd/PicoGUS-SMD.kicad_sch (KiCad schematic)
At the start: 36 parts, among them J1 2x9 header, J3 Bus_ISA_8bit, J5 SJ1-3535NG (black), J6 1x40 breakaway header, J7 1x40 breakaway header, U1 Raspberry Pi Pico, U10 74LVC2G06, U2 74LVC244, U3 SN74CB3T3257, U4 SN74CB3T3257, U5 74AHC14, U6 74LVC00, U7 74LVC1G00, U8 APS6404L-3SQR-SN

Commit message: Experimental 2nd IRQ (J10/J11), DMA label fix, labels grouped
- U2's spare channel (2A2 pin 13 -> 2Y2 pin 7, same drive and ~BUSOE as the
  IRQ output) now drives an optional second IRQ: J10 (next to the PSRAM,
  short stub on the fast SPI line) links GPIO3/SPI_TX to 2A2, R25 (10k)
  holds it low when open; J11 (next to J1) links 2Y2 to ISA IRQ3.
  GPIO3 is the PSRAM SPI_TX (all 26 Pico GPIOs are used), so this is for
  firmware that leaves the PSRAM idle. THT and SMD, ERC 0 errors.
- DMA heading moved back beside IRQ above J1.
- Silkscreen labels are members of their circuit-block KiCad groups
  (DAC, MIXER, AUDIO OUT, WT VOL, WAVEBLASTER, MIDI OUT, TX/USBPWR,
  IRQ/DMA + jumper numbers + divider, 2ND IRQ).
- Both boards re-routed: 0 DRC errors, 0 unconnected, schematic parity OK.
- BOMs: R25, J10/J11 (from the 1x40 strip), 6 jumper shunts.

Co-Authored-By: Claude Opus 5.5 <noreply@anthropic.com>
Claude-Session: https://claude.ai/code/session_011utN3x8yYUNDvkpGCEq5yD
Parts:
- added J10, J11: Jumper, Connector_PinHeader_2.54mm:PinHeader_1x02_P2.54mm_Vertical, symbol Connector_Generic:Conn_01x02
- added R25: 10k, Resistor_SMD:R_0805_2012Metric, symbol Device:R
Connections:
- net GND: now also R25.2; no longer U2.13 (2A2)
- net IRQ3: now also J11.2 (Pin_2)
- net SPI_TX: now also J10.1 (Pin_1)
- net IRQ2ND_OUT: now reaches U2.7 (2Y2)
- net IRQ2ND_OUT: now also J11.1 (Pin_1)
- new net IRQ2ND_IN: J10.2 (Pin_2), R25.1, U2.13 (2A2)
- no-connect marks 32 -> 31
Other:
- note added: "EXPERIMENTAL 2ND IRQ J10: GPIO3 (SPI_TX) drives U2 2A2 - only when the firmware leaves the PSRAM idle (no GUS mode) J11: U2 2Y2 -> ISA IRQ3. Never together with IRQ3 on J1."
