File: hw-smd/PicoGUS-SMD.kicad_sch (KiCad schematic)
At the start: 39 parts, among them J1 2x9 header, J10 Jumper, J11 Jumper, J3 Bus_ISA_8bit, J5 SJ1-3535NG (black), J6 1x40 breakaway header, J7 1x40 breakaway header, U1 Raspberry Pi Pico, U10 74LVC2G06, U2 74LVC244, U3 SN74CB3T3257, U4 SN74CB3T3257, U5 74AHC14, U6 74LVC00, U7 74LVC1G00, U8 APS6404L-3SQR-SN

Commit message: v1.3.0: drop the experimental 2nd IRQ; back-side artwork; label clean-up
- Experimental second IRQ removed from both boards: J10, J11 and R25 are gone,
  U2 pin 13 is tied to GND again and pin 7 is unconnected, as on v1.2.
  BOMs and DigiKey upload CSVs: one 10k less, 4 jumper shunts.
- Back silkscreen: the "Mila and Alisa" artwork (hw-common/art/mila-alisa.svg)
  with the dedication below it, mirrored so it reads from the back. On THT it
  is cut out 0.3 mm around every pad and hole, and the dedication sits in the
  one pad-free strip.
- Reference labels: U3/U4 horizontal under the chips; jumper labels J1/J6/J7
  upright; round capacitor labels (C1, C2, C22, C23, C32, C33) moved to free
  spots; the J3 (ISA fingers) label is hidden.
- Both boards: 0 DRC errors, 0 unconnected, schematic parity OK; ERC 0 errors.

Co-Authored-By: Claude Opus 5.5 <noreply@anthropic.com>
Claude-Session: https://claude.ai/code/session_011utN3x8yYUNDvkpGCEq5yD
Parts:
- removed J10, J11: Jumper, Connector_PinHeader_2.54mm:PinHeader_1x02_P2.54mm_Vertical, symbol Connector_Generic:Conn_01x02
- removed R25: 10k, Resistor_SMD:R_0805_2012Metric, symbol Device:R
Connections:
- net IRQ2ND_IN is gone; now on net GND: U2.13 (2A2)
- net IRQ2ND_OUT: no longer names the net of U2.7 (2Y2)
- no-connect marks 31 -> 32
Other:
- note removed: "EXPERIMENTAL 2ND IRQ J10: GPIO3 (SPI_TX) drives U2 2A2 - only when the firmware leaves the PSRAM idle (no GUS mode) J11: U2 2Y2 -> ISA IRQ3. Never together with IRQ3 on J1."

Commit message: WIP hw-smd: GY-PCM5102 module option (J10) - routing not finished
- Schematic: J10 on the DAC sheet as on the THT board (outputs to AUDIO_L/R,
  leave out U9, C12-C20, FB3, R7, R8 when the module is fitted); ERC 0 errors.
- Board: J10 placed where it is on the THT board, colliding tracks removed.
  0 DRC errors but 17 connections still unrouted - do not order from this commit.
- BOM notes and README DAC-option section.

Co-Authored-By: Claude Opus 5.5 <noreply@anthropic.com>
Claude-Session: https://claude.ai/code/session_011utN3x8yYUNDvkpGCEq5yD
Other:
- note added: "v1.3: the GY-PCM5102 module option of v1.2 (I2S_DAC1/J4) is now J10 on the DAC sheet: it feeds the Waveblaster mixer instead of U9."
- note removed: "v1.3: the GY-PCM5102 module option of v1.2 (I2S_DAC1/J4) is removed - the on-board DAC feeds the Waveblaster mixer."
Changed lines of the file:
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@@
 		)
 	)
-	(text "v1.3: the GY-PCM5102 module option of v1.2\n(I2S_DAC1/J4) is removed - the on-board DAC\nfeeds the Waveblaster mixer."
+	(text "v1.3: the GY-PCM5102 module option of v1.2\n(I2S_DAC1/J4) is now J10 on the DAC sheet: it\nfeeds the Waveblaster mixer instead of U9."
 		(exclude_from_sim no)
 		(at 223.52 104.14 0)
