File: hw-smd/audio.kicad_sch (KiCad schematic)
At the start: 13 parts, among them U9 PCM5100A

Commit message: WIP hw-smd: GY-PCM5102 module option (J10) - routing not finished
- Schematic: J10 on the DAC sheet as on the THT board (outputs to AUDIO_L/R,
  leave out U9, C12-C20, FB3, R7, R8 when the module is fitted); ERC 0 errors.
- Board: J10 placed where it is on the THT board, colliding tracks removed.
  0 DRC errors but 17 connections still unrouted - do not order from this commit.
- BOM notes and README DAC-option section.

Co-Authored-By: Claude Opus 5.5 <noreply@anthropic.com>
Claude-Session: https://claude.ai/code/session_011utN3x8yYUNDvkpGCEq5yD
Parts:
- added J10: GY-PCM5102, PiGUS library:GY-PCM5102_Module, symbol PiGUS library:GY-PCM5102
Connections:
- net AUDIO_L: now also J10.15 (LROUT)
- net AUDIO_R: now also J10.13 (ROUT)
- net BCK: now also J10.2 (BCK)
- net DIN: now also J10.3 (DIN)
- net GND: now also J10.1 (SCK), J10.12 (AGND), J10.14 (AGND), J10.5 (GND)
- net LRCK: now also J10.4 (LCK)
- net DAC_OUTL: now reaches R7.1, U9.6 (OUTL)
- net DAC_OUTR: now reaches R8.1, U9.7 (OUTR)
- new net +5V: J10.6 (VIN)
Other:
- note added: "OPTION: GY-PCM5102 module (J10) INSTEAD OF the on-board DAC. Fit EITHER U9 + C12-C20 + FB3 + R7/R8 OR the module - never both (two DAC outputs would fight). The module has its own 470R/2.2nF output filter. Module solder jumpers: H1=L H2=L H3=H H4=L."
