File: hw-smd/wavetable.kicad_sch (KiCad schematic)
At the start: 32 parts, among them J8 SJ1-3535NG-GR (green), J9 Waveblaster 2x13 male, U11 NE5532, U12 74LVC2G06

Commit message: RV1: Bourns PTD902-2020K-A103 as primary part, Alps as alternative
Schematic fields (Manufacturer/MPN/DigiKey), BOM CSVs and DigiKey upload
files (1 and 10 boards) now use the Bourns pot (PTD902-2020K-A103-ND,
426 in stock, 24 kr vs 45 kr). Alps RK09712200HA and RK0971221Z0X are
listed as alternatives; the THT LCSC column keeps C470545 (Alps) since
LCSC does not carry the Bourns part. README cost tables updated.

Co-Authored-By: Claude Opus 5.5 <noreply@anthropic.com>
Claude-Session: https://claude.ai/code/session_011utN3x8yYUNDvkpGCEq5yD
Parts:
- RV1: DigiKey 4809-RK09712200HA-ND -> PTD902-2020K-A103-ND; MPN RK09712200HA -> PTD902-2020K-A103; Manufacturer Alps Alpine -> Bourns
Changed lines of the file:
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@@
 			)
 		)
-		(property "Manufacturer" "Alps Alpine"
+		(property "Manufacturer" "Bourns"
 			(at 152.4 104.14 0)
 			(hide yes)
@@
 			)
 		)
-		(property "MPN" "RK09712200HA"
+		(property "MPN" "PTD902-2020K-A103"
 			(at 152.4 104.14 0)
 			(hide yes)
@@
 			)
 		)
-		(property "DigiKey" "4809-RK09712200HA-ND"
+		(property "DigiKey" "PTD902-2020K-A103-ND"
 			(at 152.4 104.14 0)
 			(hide yes)
@@
 			)
 		)
-		(property "Manufacturer" "Alps Alpine"
+		(property "Manufacturer" "Bourns"
 			(at 152.4 139.7 0)
 			(hide yes)
@@
 			)
 		)
-		(property "MPN" "RK09712200HA"
+		(property "MPN" "PTD902-2020K-A103"
 			(at 152.4 139.7 0)
 			(hide yes)
@@
 			)
 		)
-		(property "DigiKey" "4809-RK09712200HA-ND"
+		(property "DigiKey" "PTD902-2020K-A103-ND"
 			(at 152.4 139.7 0)
 			(hide yes)

Commit message: Mixer: +6 dB Waveblaster gain (R10/R11/R19/R20 20k, C30/C31 47p)
Waveblaster daughterboards put out about 1-1.2 Vrms full scale (DreamBlaster X2:
AK4388, 1.13 Vrms) against the PCM5100A's 2.1 Vrms, so with unity WT gain MIDI
was 5-6 dB quieter than PCM at RV1 max.

Raise the summer's feedback and PCM input resistors from 10k to 20k on both
boards: WT gain at RV1 max = 20k/10k = 2 (+6 dB), PCM 20k/20.47k (-0.2 dB, as
before). The daughterboard load (about 4.8k at RV1 max) and the pot taper stay
unchanged. C30/C31 100p -> 47p keeps the feedback pole at ~170 kHz.

BOM-only change (no copper change): schematic values/fields, PCB values,
BOM-THT/BOM-SMD lines with the previous values in the notes, DigiKey upload
files (1x/10x), schematic PDFs. SMD C30/C31 get an LCSC field (C14857,
CL21C470JBANNNC) because DigiKey only stocks the 100 V CL21C470JC61PNC.
README mixer text updated; the THT diagram now shows R14 on the J9 side of C22
and R12 joined to the summing node. ERC 0, DRC 0 with schematic parity.

Co-Authored-By: Claude Opus 5.5 <noreply@anthropic.com>
Claude-Session: https://claude.ai/code/session_011utN3x8yYUNDvkpGCEq5yD
Parts:
- C30, C31: value 100pF C0G -> 47pF C0G; DigiKey 1276-1014-1-ND -> 1276-6521-1-ND; LCSC (none) -> C14857; MPN CL21C101JBANNNC -> CL21C470JC61PNC
- R10, R11, R19, R20: value 10k -> 20k; DigiKey YAG1763CT-ND -> YAG1823CT-ND; MPN RT0805BRD0710KL -> RT0805BRD0720KL
Changed lines of the file:
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@@
 			)
 		)
-		(property "Value" "10k"
+		(property "Value" "20k"
 			(at 167.64 93.98 90)
 			(show_name no)
@@
 			)
 		)
-		(property "MPN" "RT0805BRD0710KL"
+		(property "MPN" "RT0805BRD0720KL"
 			(at 167.64 91.44 0)
 			(hide yes)
@@
 			)
 		)
-		(property "DigiKey" "YAG1763CT-ND"
+		(property "DigiKey" "YAG1823CT-ND"
 			(at 167.64 91.44 0)
 			(hide yes)
@@
 			)
 		)
-		(property "Value" "10k"
+		(property "Value" "20k"
 			(at 193.04 88.04 90)
 			(show_name no)
@@
 			)
 		)
-		(property "MPN" "RT0805BRD0710KL"
+		(property "MPN" "RT0805BRD0720KL"
 			(at 187.96 86.36 0)
 			(hide yes)
@@
 			)
 		)
-		(property "DigiKey" "YAG1763CT-ND"
+		(property "DigiKey" "YAG1823CT-ND"
 			(at 187.96 86.36 0)
 			(hide yes)
@@
 			)
 		)
-		(property "Value" "100pF C0G"
+		(property "Value" "47pF C0G"
 			(at 186.69 77.47 90)
 			(show_name no)
@@
 			)
 		)
-		(property "MPN" "CL21C101JBANNNC"
+		(property "MPN" "CL21C470JC61PNC"
 			(at 187.96 81.28 0)
 			(hide yes)
@@
 			)
 		)
-		(property "DigiKey" "1276-1014-1-ND"
+		(property "DigiKey" "1276-6521-1-ND"
+			(at 187.96 81.28 0)
+			(hide yes)
+			(show_name no)
+			(do_not_autoplace no)
+			(effects
+				(font
+					(size 1.27 1.27)
+				)
+			)
+		)
+		(property "LCSC" "C14857"
 			(at 187.96 81.28 0)
 			(hide yes)
@@
 			)
 		)
-		(property "Value" "10k"
+		(property "Value" "20k"
 			(at 167.64 129.54 90)
 			(show_name no)
@@
 			)
 		)
-		(property "MPN" "RT0805BRD0710KL"
+		(property "MPN" "RT0805BRD0720KL"
 			(at 167.64 127 0)
 			(hide yes)
@@
 			)
 		)
-		(property "DigiKey" "YAG1763CT-ND"
+		(property "DigiKey" "YAG1823CT-ND"
 			(at 167.64 127 0)
 			(hide yes)
@@
 			)
 		)
-		(property "Value" "10k"
+		(property "Value" "20k"
 			(at 193.04 123.6 90)
 			(show_name no)
@@
 			)
 		)
-		(property "MPN" "RT0805BRD0710KL"
+		(property "MPN" "RT0805BRD0720KL"
 			(at 187.96 121.92 0)
 			(hide yes)
@@
 			)
 		)
-		(property "DigiKey" "YAG1763CT-ND"
+		(property "DigiKey" "YAG1823CT-ND"
 			(at 187.96 121.92 0)
 			(hide yes)
@@
 			)
 		)
-		(property "Value" "100pF C0G"
+		(property "Value" "47pF C0G"
 			(at 186.69 113.03 90)
 			(show_name no)
@@
 			)
 		)
-		(property "MPN" "CL21C101JBANNNC"
+		(property "MPN" "CL21C470JC61PNC"
 			(at 187.96 116.84 0)
 			(hide yes)
@@
 			)
 		)
-		(property "DigiKey" "1276-1014-1-ND"
+		(property "DigiKey" "1276-6521-1-ND"
 			(at 187.96 116.84 0)
 			(hide yes)
+			(show_name no)
+			(do_not_autoplace no)
+			(effects
+				(font
+					(size 1.27 1.27)
+				)
+			)
+		)
+		(property "LCSC" "C14857"
+			(at 187.96 116.84 0)
+			(hide yes)
