File: hw-tht/PicoGUS-THT.kicad_sch (KiCad schematic)
At the start: 38 parts, among them J1 IRQDMA_JP, J3 Bus_ISA_8bit, J5 SJ1-3535NG, J6 UART_TX, J7 USB power jumper, U1 Pico, U10 74AHCT126, U2 74AHC244, U3 SN74CB3T3257, U4 SN74CB3T3257, U5 74AHC14, U6 74AHC00, U7 74AHC00, U8 APS6404L-3SQR-SN

Commit message: hw-tht: cleaner audio supplies, bipolar WT coupling caps, circuit-block groups
- DAC AVDD (U9 pin 8) gets its own rail behind ferrite bead FB3, with C13/C15
  at the pin; DVDD/CPVDD stay on the Pico 3V3.
- NE5532 +/-12 V from ISA through R23/R24 (10R) + C32/C33 (47uF) RC filters,
  C28/C29 0.1uF stay at the op-amp pins.
- C22/C23 WT coupling caps are now 10uF bipolar (Panasonic ECE-A1HN100U):
  the DC across them depends on the daughterboard.
- Every chip and its decoupling caps/resistors form a KiCad group.
- DAC pre-routes reworked (VNEG via B.Cu, XSMT via); RUN RC moved out of the
  Pico fan-in. Fully routed, 0 DRC errors, 0 unconnected.
- BOM: new lines for R23/R24, FB3, C32/C33; README has DigiKey cost in NOK.

Co-Authored-By: Claude Opus 5.5 <noreply@anthropic.com>
Claude-Session: https://claude.ai/code/session_011utN3x8yYUNDvkpGCEq5yD
Parts:
- FB1, FB2: Alternatives Fair-Rite 2761001112 (DK 1934-1423-1-ND, 33346). A wire link also works (slightly worse EMI). -> Fair-Rite 2761001112 (DK 1934-1423-1-ND, 33346). A wire link also works (slightly worse EMI / DAC noise).
Changed lines of the file:
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@@
 			)
 		)
-		(property "Description" "47uF 16V aluminium electrolytic, 5mm dia, 2mm pitch"
+		(property "Description" "47uF 35V aluminium electrolytic, 5mm dia, 2mm pitch"
 			(at 67.945 186.69 0)
 			(hide yes)
@@
 			)
 		)
-		(property "Description" "47uF 16V aluminium electrolytic, 5mm dia, 2mm pitch"
+		(property "Description" "47uF 35V aluminium electrolytic, 5mm dia, 2mm pitch"
 			(at 20.955 186.69 0)
 			(hide yes)
@@
 			)
 		)
-		(property "Description" "Axial ferrite bead (bead on leads), MIDI out EMI filter"
+		(property "Description" "Axial ferrite bead (bead on leads): MIDI out EMI filter, DAC AVDD filter"
 			(at 232.41 70.485 0)
 			(hide yes)
@@
 			)
 		)
-		(property "Alternatives" "Fair-Rite 2761001112 (DK 1934-1423-1-ND, 33346). A wire link also works (slightly worse EMI)."
+		(property "Alternatives" "Fair-Rite 2761001112 (DK 1934-1423-1-ND, 33346). A wire link also works (slightly worse EMI / DAC noise)."
 			(at 232.41 70.485 0)
 			(hide yes)
@@
 			)
 		)
-		(property "Description" "Axial ferrite bead (bead on leads), MIDI out EMI filter"
+		(property "Description" "Axial ferrite bead (bead on leads): MIDI out EMI filter, DAC AVDD filter"
 			(at 240.03 60.325 0)
 			(hide yes)
@@
 			)
 		)
-		(property "Alternatives" "Fair-Rite 2761001112 (DK 1934-1423-1-ND, 33346). A wire link also works (slightly worse EMI)."
+		(property "Alternatives" "Fair-Rite 2761001112 (DK 1934-1423-1-ND, 33346). A wire link also works (slightly worse EMI / DAC noise)."
 			(at 240.03 60.325 0)
 			(hide yes)

Commit message: hw-tht: PWR_FLAG on Pico VBUS, ERC now 0 errors
VBUS is fed from the Pico's USB socket or through the USBPWR jumper J7,
so nothing on the schematic drives it (same ERC error on v1.2).
Schematic only, the PCB is unchanged.

Co-Authored-By: Claude Opus 5.5 <noreply@anthropic.com>
Claude-Session: https://claude.ai/code/session_011utN3x8yYUNDvkpGCEq5yD
Changed lines of the file:
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@@
+		)
+	)
+	(symbol
+		(lib_id "power:PWR_FLAG")
+		(at 127 31.115 0)
+		(unit 1)
+		(body_style 1)
+		(exclude_from_sim no)
+		(in_bom no)
+		(on_board yes)
+		(in_pos_files no)
+		(dnp no)
+		(property "Reference" "#FLG102"
+			(at 127 31.115 0)
+			(hide yes)
+			(show_name no)
+			(do_not_autoplace no)
+			(effects
+				(font
+					(size 1.27 1.27)
+				)
+			)
+		)
+		(property "Value" "PWR_FLAG"
+			(at 127 27.305 0)
+			(show_name no)
+			(do_not_autoplace no)
+			(effects
+				(font
+					(size 1.27 1.27)
+				)
+			)
+		)
+		(property "Footprint" ""
+			(at 127 31.115 0)
+			(hide yes)
+			(show_name no)
+			(do_not_autoplace no)
+			(effects
+				(font
+					(size 1.27 1.27)
+				)
+			)
+		)
+		(property "Datasheet" ""
+			(at 127 31.115 0)
+			(hide yes)
+			(show_name no)
+			(do_not_autoplace no)
+			(effects
+				(font
+					(size 1.27 1.27)
+				)
+			)
+		)
+		(property "Description" ""
+			(at 127 31.115 0)
+			(hide yes)
+			(show_name no)
+			(do_not_autoplace no)
+			(effects
+				(font
+					(size 1.27 1.27)
+				)
+			)
+		)
+		(pin "1"
+		)
+		(instances
+			(project "PicoGUS-THT"
+				(path "/8fb4b197-630e-4faa-9892-8ecaeb71c13b"
+					(reference "#FLG102")
+					(unit 1)
+				)
+			)
 		)
 	)

Commit message: hw-tht: GY-PCM5102 module option (J10) as an either/or alternative to the DAC
- J10 (new footprint PiGUS library:GY-PCM5102_Module + symbol): the module plugs
  in on female headers - its I2S row (SCK->GND, BCK, DIN, LCK, GND, VIN=+5V) and
  the AGND/ROUT/AGND/LROUT end of its 9-pin row, as I2S_DAC1/J4 on v1.2. Its
  outputs join U9's (DAC_OUTL/R) ahead of R7/R8 + C19/C20, so the mixer, WT path
  and firmware are unchanged. Fit U9 + C12-C18 + FB3 OR the module, never both.
- Placed right of the Waveblaster area over low parts (courtyard only around the
  pins); R4 and C28 moved a few mm. Oval pads keep two tracks per gap.
- Silkscreen: dashed "DAC" outline around the parts to leave out for the module
  (R7/R8 notched out: they stay), heading "DAC -OR- J10 MODULE", dashed module
  outline labelled "J10: GY-PCM5102".
- BOM: J10 module + 1x6/1x4 female headers as optional lines; U9 note.
- README: DAC option section with the fit/leave-out table.
- Re-routed around the module: 0 DRC errors, 0 unconnected, schematic parity OK;
  ERC 0 errors.

Co-Authored-By: Claude Opus 5.5 <noreply@anthropic.com>
Claude-Session: https://claude.ai/code/session_011utN3x8yYUNDvkpGCEq5yD
Other:
- note added: "THT board: the GY-PCM5102 module option of v1.2 (I2S_DAC1/J4) is now J10 on the DAC sheet: it feeds the Waveblaster mixer instead of U9."
- note removed: "THT board: the GY-PCM5102 module option of v1.2 (I2S_DAC1/J4) is removed - the on-board DAC feeds the Waveblaster mixer."
Changed lines of the file:
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@@
 		)
 	)
-	(text "THT board: the GY-PCM5102 module option of v1.2\n(I2S_DAC1/J4) is removed - the on-board DAC\nfeeds the Waveblaster mixer."
+	(text "THT board: the GY-PCM5102 module option of v1.2\n(I2S_DAC1/J4) is now J10 on the DAC sheet: it\nfeeds the Waveblaster mixer instead of U9."
 		(exclude_from_sim no)
 		(at 223.52 104.14 0)
