File: hw-tht/wavetable.kicad_sch (KiCad schematic)
At the start: 29 parts, among them J8 SJ1-3535NG-GR, J9 Waveblaster, U10 74AHCT126, U11 NE5532, U7 74AHC00

Commit message: hw-tht: v1.3.0, axial/0805 hybrid resistors, decoupling placement
- Board revision v1.3.0 (schematic title blocks and README); take over
  the reviewed layout including the rotated PicoGUS logo and the new
  version and credit texts. The review board is now the build base, so
  its artwork is kept as drawn.
- New R_Axial_DIN0207_P10.16mm_0805_Hybrid footprint (0805 pads between
  the axial holes) for all resistors; BOM lists Yageo RC0805 (DigiKey)
  and UNI-ROYAL 0805W8F (LCSC) alternatives.
- Decoupling back next to the pins it serves, as on v1.2: DAC caps at
  CPVDD/CAPP-CAPM/VNEG/AVDD/DVDD, C4 at U2, C10 at the PSRAM, C3/C5 on
  the supply side of U3/U4. MIDI resistors and ferrites in one row
  next to J5, DAC output filters below the DAC.

Co-Authored-By: Claude Opus 5.5 <noreply@anthropic.com>
Claude-Session: https://claude.ai/code/session_011utN3x8yYUNDvkpGCEq5yD
Parts:
- R10, R11, R12, R13, R16, R19, R20, R9: footprint Resistor_THT:R_Axial_DIN0207_L6.3mm_D2.5mm_P10.16mm_Horizontal -> PicoGUS-THT:R_Axial_DIN0207_P10.16mm_0805_Hybrid; Alternatives (none) -> 0805 SMD (fits between the holes): Yageo RC0805FR-0710KL (D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
- R14, R15: footprint Resistor_THT:R_Axial_DIN0207_L6.3mm_D2.5mm_P10.16mm_Horizontal -> PicoGUS-THT:R_Axial_DIN0207_P10.16mm_0805_Hybrid; Alternatives (none) -> 0805 SMD (fits between the holes): Yageo RC0805FR-07100KL (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
- R21, R22: footprint Resistor_THT:R_Axial_DIN0207_L6.3mm_D2.5mm_P10.16mm_Horizontal -> PicoGUS-THT:R_Axial_DIN0207_P10.16mm_0805_Hybrid; Alternatives (none) -> 0805 SMD (fits between the holes): Yageo RC0805FR-07100RL (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
Changed lines of the file:
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@@
 		(title "PicoGUS THT - Waveblaster header & line-out mixer")
 		(date "2026-09-28")
-		(rev "v1.2-THT")
+		(rev "v1.3.0")
 		(comment 1 "Waveblaster (wavetable) daughterboard header, analog WT volume and op-amp mixer")
 		(comment 2 "Derived from the hand386 ISA adapter mixer and the PicoGUS 2.0 WT header")
@@
 			)
 		)
-		(property "Footprint" "Resistor_THT:R_Axial_DIN0207_L6.3mm_D2.5mm_P10.16mm_Horizontal"
+		(property "Footprint" "PicoGUS-THT:R_Axial_DIN0207_P10.16mm_0805_Hybrid"
 			(at 133.35 38.1 0)
 			(hide yes)
@@
 			)
 		)
+		(property "Alternatives" "0805 SMD (fits between the holes): Yageo RC0805FR-0710KL (DK 311-10.0KCRCT-ND, 2120333), UNI-ROYAL 0805W8F (LCSC C17414, 43352900)."
+			(at 133.35 38.1 0)
+			(hide yes)
+			(show_name no)
+			(do_not_autoplace no)
+			(effects
+				(font
+					(size 1.27 1.27)
+				)
+			)
+		)
 		(pin "1"
 		)
@@
 			)
 		)
-		(property "Footprint" "Resistor_THT:R_Axial_DIN0207_L6.3mm_D2.5mm_P10.16mm_Horizontal"
+		(property "Footprint" "PicoGUS-THT:R_Axial_DIN0207_P10.16mm_0805_Hybrid"
 			(at 133.35 63.5 0)
 			(hide yes)
@@
 			)
 		)
+		(property "Alternatives" "0805 SMD (fits between the holes): Yageo RC0805FR-0710KL (DK 311-10.0KCRCT-ND, 2120333), UNI-ROYAL 0805W8F (LCSC C17414, 43352900)."
+			(at 133.35 63.5 0)
+			(hide yes)
+			(show_name no)
+			(do_not_autoplace no)
+			(effects
+				(font
+					(size 1.27 1.27)
+				)
+			)
+		)
 		(pin "1"
 		)
@@
 			)
 		)
-		(property "Footprint" "Resistor_THT:R_Axial_DIN0207_L6.3mm_D2.5mm_P10.16mm_Horizontal"
+		(property "Footprint" "PicoGUS-THT:R_Axial_DIN0207_P10.16mm_0805_Hybrid"
 			(at 167.64 91.44 0)
 			(hide yes)
@@
 			)
 		)
+		(property "Alternatives" "0805 SMD (fits between the holes): Yageo RC0805FR-0710KL (DK 311-10.0KCRCT-ND, 2120333), UNI-ROYAL 0805W8F (LCSC C17414, 43352900)."
+			(at 167.64 91.44 0)
+			(hide yes)
+			(show_name no)
+			(do_not_autoplace no)
+			(effects
+				(font
+					(size 1.27 1.27)
+				)
+			)
+		)
 		(pin "1"
 		)
@@
 			)
 		)
-		(property "Footprint" "Resistor_THT:R_Axial_DIN0207_L6.3mm_D2.5mm_P10.16mm_Horizontal"
+		(property "Footprint" "PicoGUS-THT:R_Axial_DIN0207_P10.16mm_0805_Hybrid"
 			(at 187.96 86.36 0)
 			(hide yes)
@@
 			)
 		)
+		(property "Alternatives" "0805 SMD (fits between the holes): Yageo RC0805FR-0710KL (DK 311-10.0KCRCT-ND, 2120333), UNI-ROYAL 0805W8F (LCSC C17414, 43352900)."
+			(at 187.96 86.36 0)
+			(hide yes)
+			(show_name no)
+			(do_not_autoplace no)
+			(effects
+				(font
+					(size 1.27 1.27)
+				)
+			)
+		)
 		(pin "1"
 		)
@@
 			)
 		)
-		(property "Footprint" "Resistor_THT:R_Axial_DIN0207_L6.3mm_D2.5mm_P10.16mm_Horizontal"
+		(property "Footprint" "PicoGUS-THT:R_Axial_DIN0207_P10.16mm_0805_Hybrid"
 			(at 203.2 93.98 0)
 			(hide yes)
@@
 			)
 		)
+		(property "Alternatives" "0805 SMD (fits between the holes): Yageo RC0805FR-07100RL (DK 311-100CRCT-ND, 1562462), UNI-ROYAL 0805W8F (LCSC C17408, 7823800)."
+			(at 203.2 93.98 0)
+			(hide yes)
+			(show_name no)
+			(do_not_autoplace no)
+			(effects
+				(font
+					(size 1.27 1.27)
+				)
+			)
+		)
 		(pin "1"
 		)
@@
 			)
 		)
-		(property "Footprint" "Resistor_THT:R_Axial_DIN0207_L6.3mm_D2.5mm_P10.16mm_Horizontal"
+		(property "Footprint" "PicoGUS-THT:R_Axial_DIN0207_P10.16mm_0805_Hybrid"
 			(at 135.89 104.14 0)
 			(hide yes)
@@
 			)
 		)
+		(property "Alternatives" "0805 SMD (fits between the holes): Yageo RC0805FR-07100KL (DK 311-100KCRCT-ND, 1068493), UNI-ROYAL 0805W8F (LCSC C149504, 3119100)."
+			(at 135.89 104.14 0)
+			(hide yes)
+			(show_name no)
+			(do_not_autoplace no)
+			(effects
+				(font
+					(size 1.27 1.27)
+				)
+			)
+		)
 		(pin "1"
 		)
@@
 			)
 		)
-		(property "Footprint" "Resistor_THT:R_Axial_DIN0207_L6.3mm_D2.5mm_P10.16mm_Horizontal"
+		(property "Footprint" "PicoGUS-THT:R_Axial_DIN0207_P10.16mm_0805_Hybrid"
 			(at 167.64 104.14 0)
 			(hide yes)
@@
 			)
 		)
+		(property "Alternatives" "0805 SMD (fits between the holes): Yageo RC0805FR-0710KL (DK 311-10.0KCRCT-ND, 2120333), UNI-ROYAL 0805W8F (LCSC C17414, 43352900)."
+			(at 167.64 104.14 0)
+			(hide yes)
+			(show_name no)
+			(do_not_autoplace no)
+			(effects
+				(font
+					(size 1.27 1.27)
+				)
+			)
+		)
 		(pin "1"
 		)
@@
 			)
 		)
-		(property "Footprint" "Resistor_THT:R_Axial_DIN0207_L6.3mm_D2.5mm_P10.16mm_Horizontal"
+		(property "Footprint" "PicoGUS-THT:R_Axial_DIN0207_P10.16mm_0805_Hybrid"
 			(at 167.64 127 0)
 			(hide yes)
@@
 			)
 		)
+		(property "Alternatives" "0805 SMD (fits between the holes): Yageo RC0805FR-0710KL (DK 311-10.0KCRCT-ND, 2120333), UNI-ROYAL 0805W8F (LCSC C17414, 43352900)."
+			(at 167.64 127 0)
+			(hide yes)
+			(show_name no)
+			(do_not_autoplace no)
+			(effects
+				(font
+					(size 1.27 1.27)
+				)
+			)
+		)
 		(pin "1"
 		)
@@
 			)
 		)
-		(property "Footprint" "Resistor_THT:R_Axial_DIN0207_L6.3mm_D2.5mm_P10.16mm_Horizontal"
+		(property "Footprint" "PicoGUS-THT:R_Axial_DIN0207_P10.16mm_0805_Hybrid"
 			(at 187.96 121.92 0)
 			(hide yes)
@@
 			)
 		)
+		(property "Alternatives" "0805 SMD (fits between the holes): Yageo RC0805FR-0710KL (DK 311-10.0KCRCT-ND, 2120333), UNI-ROYAL 0805W8F (LCSC C17414, 43352900)."
+			(at 187.96 121.92 0)
+			(hide yes)
+			(show_name no)
+			(do_not_autoplace no)
+			(effects
+				(font
+					(size 1.27 1.27)
+				)
+			)
+		)
 		(pin "1"
 		)
@@
 			)
 		)
-		(property "Footprint" "Resistor_THT:R_Axial_DIN0207_L6.3mm_D2.5mm_P10.16mm_Horizontal"
+		(property "Footprint" "PicoGUS-THT:R_Axial_DIN0207_P10.16mm_0805_Hybrid"
 			(at 203.2 129.54 0)
 			(hide yes)
@@
 			)
 		)
+		(property "Alternatives" "0805 SMD (fits between the holes): Yageo RC0805FR-07100RL (DK 311-100CRCT-ND, 1562462), UNI-ROYAL 0805W8F (LCSC C17408, 7823800)."
+			(at 203.2 129.54 0)
+			(hide yes)
+			(show_name no)
+			(do_not_autoplace no)
+			(effects
+				(font
+					(size 1.27 1.27)
+				)
+			)
+		)
 		(pin "1"
 		)
@@
 			)
 		)
-		(property "Footprint" "Resistor_THT:R_Axial_DIN0207_L6.3mm_D2.5mm_P10.16mm_Horizontal"
+		(property "Footprint" "PicoGUS-THT:R_Axial_DIN0207_P10.16mm_0805_Hybrid"
 			(at 135.89 139.7 0)
 			(hide yes)
@@
 			)
 		)
+		(property "Alternatives" "0805 SMD (fits between the holes): Yageo RC0805FR-07100KL (DK 311-100KCRCT-ND, 1068493), UNI-ROYAL 0805W8F (LCSC C149504, 3119100)."
+			(at 135.89 139.7 0)
+			(hide yes)
+			(show_name no)
+			(do_not_autoplace no)
+			(effects
+				(font
+					(size 1.27 1.27)
+				)
+			)
+		)
 		(pin "1"
 		)
@@
 			)
 		)
-		(property "Footprint" "Resistor_THT:R_Axial_DIN0207_L6.3mm_D2.5mm_P10.16mm_Horizontal"
+		(property "Footprint" "PicoGUS-THT:R_Axial_DIN0207_P10.16mm_0805_Hybrid"
 			(at 167.64 139.7 0)
 			(hide yes)
@@
 			(at 167.64 139.7 0)
 			(hide yes)
+			(show_name no)
+			(do_not_autoplace no)
+			(effects
+				(font
+					(size 1.27 1.27)
+				)
+			)
+		)
+		(property "Alternatives" "0805 SMD (fits between the holes): Yageo RC0805FR-0710KL (DK 311-10.0KCRCT-ND, 2120333), UNI-ROYAL 0805W8F (LCSC C17414, 43352900)."
+			(at 167.64 139.7 0)
+			(hide yes)

Commit message: hw-tht: 5 mm disc/0805 hybrid capacitors, labels inside or beside bodies
- New C_Disc_D5.0mm_W2.5mm_P5.00mm_0805_Hybrid footprint for all ceramic
  caps: 5.0/5.08 mm radial part OR an 0805 between the holes. Replaces
  the 2.5/5.0 mm dual-pitch footprint.
- BOM: every ceramic cap line is now 5 mm pitch at both distributors
  (2.2 nF LCSC Dersonic C22391154, 100 pF DigiKey Vishay
  K101J15C0GF5TH5) and lists an in-stock 0805 alternative.
- Silkscreen labels: FB1/FB2 inside the body like the resistors;
  capacitor labels just outside the body, above/left, else at a free end.

Co-Authored-By: Claude Opus 5.5 <noreply@anthropic.com>
Claude-Session: https://claude.ai/code/session_011utN3x8yYUNDvkpGCEq5yD
Parts:
- C21, C25, C26, C27, C28, C29: footprint PicoGUS-THT:C_Disc_D5.0mm_W2.5mm_P2.50mm_P5.00mm -> PicoGUS-THT:C_Disc_D5.0mm_W2.5mm_P5.00mm_0805_Hybrid; Alternatives (none) -> 0805 SMD (fits between the holes): Samsung CL21B104KBCNNNC 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
- C24: footprint PicoGUS-THT:C_Disc_D5.0mm_W2.5mm_P2.50mm_P5.00mm -> PicoGUS-THT:C_Disc_D5.0mm_W2.5mm_P5.00mm_0805_Hybrid; Alternatives (none) -> 0805 SMD 25V X5R: Taiyo Yuden EMK212BJ106KG-T (DK 587-1295-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
- C30, C31: footprint PicoGUS-THT:C_Disc_D5.0mm_W2.5mm_P2.50mm_P5.00mm -> PicoGUS-THT:C_Disc_D5.0mm_W2.5mm_P5.00mm_0805_Hybrid; Alternatives (none) -> THT: TDK FG28C0G1H101JNT06 (DK 445-173472-1-ND). 0805 SMD: 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; DigiKey 399-C320C101J5G5TA-ND -> BC1042CT-ND; MPN C320C101J5G5TA -> K101J15C0GF5TH5; Manufacturer KEMET -> Vishay
Changed lines of the file:
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@@
 			)
 		)
-		(property "Footprint" "PicoGUS-THT:C_Disc_D5.0mm_W2.5mm_P2.50mm_P5.00mm"
+		(property "Footprint" "PicoGUS-THT:C_Disc_D5.0mm_W2.5mm_P5.00mm_0805_Hybrid"
 			(at 40.64 127 0)
 			(hide yes)
@@
 			)
 		)
+		(property "Alternatives" "0805 SMD 25V X5R: Taiyo Yuden EMK212BJ106KG-T (DK 587-1295-1-ND, 1864) or Samsung CL21A106KAYNNNE (LCSC C15850, 878060)."
+			(at 40.64 127 0)
+			(hide yes)
+			(show_name no)
+			(do_not_autoplace no)
+			(effects
+				(font
+					(size 1.27 1.27)
+				)
+			)
+		)
 		(pin "1"
 		)
@@
 			)
 		)
-		(property "Footprint" "PicoGUS-THT:C_Disc_D5.0mm_W2.5mm_P2.50mm_P5.00mm"
+		(property "Footprint" "PicoGUS-THT:C_Disc_D5.0mm_W2.5mm_P5.00mm_0805_Hybrid"
 			(at 48.26 127 0)
 			(hide yes)
@@
 			)
 		)
+		(property "Alternatives" "0805 SMD (fits between the holes): Samsung CL21B104KBCNNNC (DK 1276-1003-1-ND, 4889645; LCSC C1711, 1029920)."
+			(at 48.26 127 0)
+			(hide yes)
+			(show_name no)
+			(do_not_autoplace no)
+			(effects
+				(font
+					(size 1.27 1.27)
+				)
+			)
+		)
 		(pin "1"
 		)
@@
 			)
 		)
-		(property "Footprint" "PicoGUS-THT:C_Disc_D5.0mm_W2.5mm_P2.50mm_P5.00mm"
+		(property "Footprint" "PicoGUS-THT:C_Disc_D5.0mm_W2.5mm_P5.00mm_0805_Hybrid"
 			(at 55.88 127 0)
 			(hide yes)
@@
 			)
 		)
+		(property "Alternatives" "0805 SMD (fits between the holes): Samsung CL21B104KBCNNNC (DK 1276-1003-1-ND, 4889645; LCSC C1711, 1029920)."
+			(at 55.88 127 0)
+			(hide yes)
+			(show_name no)
+			(do_not_autoplace no)
+			(effects
+				(font
+					(size 1.27 1.27)
+				)
+			)
+		)
 		(pin "1"
 		)
@@
 			)
 		)
-		(property "Footprint" "PicoGUS-THT:C_Disc_D5.0mm_W2.5mm_P2.50mm_P5.00mm"
+		(property "Footprint" "PicoGUS-THT:C_Disc_D5.0mm_W2.5mm_P5.00mm_0805_Hybrid"
 			(at 63.5 127 0)
 			(hide yes)
@@
 			)
 		)
+		(property "Alternatives" "0805 SMD (fits between the holes): Samsung CL21B104KBCNNNC (DK 1276-1003-1-ND, 4889645; LCSC C1711, 1029920)."
+			(at 63.5 127 0)
+			(hide yes)
+			(show_name no)
+			(do_not_autoplace no)
+			(effects
+				(font
+					(size 1.27 1.27)
+				)
+			)
+		)
 		(pin "1"
 		)
@@
 			)
 		)
-		(property "Footprint" "PicoGUS-THT:C_Disc_D5.0mm_W2.5mm_P2.50mm_P5.00mm"
+		(property "Footprint" "PicoGUS-THT:C_Disc_D5.0mm_W2.5mm_P5.00mm_0805_Hybrid"
 			(at 124.46 142.24 0)
 			(hide yes)
@@
 			)
 		)
+		(property "Alternatives" "0805 SMD (fits between the holes): Samsung CL21B104KBCNNNC (DK 1276-1003-1-ND, 4889645; LCSC C1711, 1029920)."
+			(at 124.46 142.24 0)
+			(hide yes)
+			(show_name no)
+			(do_not_autoplace no)
+			(effects
+				(font
+					(size 1.27 1.27)
+				)
+			)
+		)
 		(pin "1"
 		)
@@
 			)
 		)
-		(property "Footprint" "PicoGUS-THT:C_Disc_D5.0mm_W2.5mm_P2.50mm_P5.00mm"
+		(property "Footprint" "PicoGUS-THT:C_Disc_D5.0mm_W2.5mm_P5.00mm_0805_Hybrid"
 			(at 187.96 81.28 0)
 			(hide yes)
@@
 			)
 		)
-		(property "Manufacturer" "KEMET"
+		(property "Manufacturer" "Vishay"
 			(at 187.96 81.28 0)
 			(hide yes)
@@
 			)
 		)
-		(property "MPN" "C320C101J5G5TA"
+		(property "MPN" "K101J15C0GF5TH5"
 			(at 187.96 81.28 0)
 			(hide yes)
@@
 			)
 		)
-		(property "DigiKey" "399-C320C101J5G5TA-ND"
+		(property "DigiKey" "BC1042CT-ND"
 			(at 187.96 81.28 0)
 			(hide yes)
@@
 			)
 		)
+		(property "Alternatives" "THT: TDK FG28C0G1H101JNT06 (DK 445-173472-1-ND). 0805 SMD: Samsung CL21C101JBANNNC (DK 1276-1014-1-ND, 104603; LCSC C1790, 186200)."
+			(at 187.96 81.28 0)
+			(hide yes)
+			(show_name no)
+			(do_not_autoplace no)
+			(effects
+				(font
+					(size 1.27 1.27)
+				)
+			)
+		)
 		(pin "1"
 		)
@@
 			)
 		)
-		(property "Footprint" "PicoGUS-THT:C_Disc_D5.0mm_W2.5mm_P2.50mm_P5.00mm"
+		(property "Footprint" "PicoGUS-THT:C_Disc_D5.0mm_W2.5mm_P5.00mm_0805_Hybrid"
 			(at 187.96 116.84 0)
 			(hide yes)
@@
 			)
 		)
-		(property "Manufacturer" "KEMET"
+		(property "Manufacturer" "Vishay"
 			(at 187.96 116.84 0)
 			(hide yes)
@@
 			)
 		)
-		(property "MPN" "C320C101J5G5TA"
+		(property "MPN" "K101J15C0GF5TH5"
 			(at 187.96 116.84 0)
 			(hide yes)
@@
 			)
 		)
-		(property "DigiKey" "399-C320C101J5G5TA-ND"
+		(property "DigiKey" "BC1042CT-ND"
 			(at 187.96 116.84 0)
 			(hide yes)
@@
 			)
 		)
+		(property "Alternatives" "THT: TDK FG28C0G1H101JNT06 (DK 445-173472-1-ND). 0805 SMD: Samsung CL21C101JBANNNC (DK 1276-1014-1-ND, 104603; LCSC C1790, 186200)."
+			(at 187.96 116.84 0)
+			(hide yes)
+			(show_name no)
+			(do_not_autoplace no)
+			(effects
+				(font
+					(size 1.27 1.27)
+				)
+			)
+		)
 		(pin "1"
 		)
@@
 			)
 		)
-		(property "Footprint" "PicoGUS-THT:C_Disc_D5.0mm_W2.5mm_P2.50mm_P5.00mm"
+		(property "Footprint" "PicoGUS-THT:C_Disc_D5.0mm_W2.5mm_P5.00mm_0805_Hybrid"
 			(at 250.19 88.9 0)
 			(hide yes)
@@
 			)
 		)
+		(property "Alternatives" "0805 SMD (fits between the holes): Samsung CL21B104KBCNNNC (DK 1276-1003-1-ND, 4889645; LCSC C1711, 1029920)."
+			(at 250.19 88.9 0)
+			(hide yes)
+			(show_name no)
+			(do_not_autoplace no)
+			(effects
+				(font
+					(size 1.27 1.27)
+				)
+			)
+		)
 		(pin "1"
 		)
@@
 			)
 		)
-		(property "Footprint" "PicoGUS-THT:C_Disc_D5.0mm_W2.5mm_P2.50mm_P5.00mm"
+		(property "Footprint" "PicoGUS-THT:C_Disc_D5.0mm_W2.5mm_P5.00mm_0805_Hybrid"
 			(at 260.35 88.9 0)
 			(hide yes)
@@
 			(at 260.35 88.9 0)
 			(hide yes)
+			(show_name no)
+			(do_not_autoplace no)
+			(effects
+				(font
+					(size 1.27 1.27)
+				)
+			)
+		)
+		(property "Alternatives" "0805 SMD (fits between the holes): Samsung CL21B104KBCNNNC (DK 1276-1003-1-ND, 4889645; LCSC C1711, 1029920)."
+			(at 260.35 88.9 0)
+			(hide yes)

Commit message: hw-tht: through-hole parts only, drop the hybrid footprints
- Resistors: plain axial DIN0207 (10.16 mm); ceramic caps: plain 5 mm
  disc; FB1/FB2: axial bead on leads (12.7 mm, Fair-Rite 2743002112 /
  LCSC FH RH3.5x0.8x9P52E); logic ICs: plain DIP-14/DIP-20.
- Only the parts that have no THT version stay SMD: U3/U4 (CB3T3257),
  U8 (APS6404L PSRAM), U9 (PCM510x DAC).
- BOM: 0805/TSSOP alternatives removed. The DIP logic ICs are DigiKey
  parts; LCSC has almost none in stock (listed with their real stock).
- Placement from the latest layout review (DIPs in one column, DAC and
  its caps next to the bus switches), FB1/FB2 and C19/C20 shifted to fit
  the longer bead footprint. Passive labels centred inside the bodies.

Co-Authored-By: Claude Opus 5.5 <noreply@anthropic.com>
Claude-Session: https://claude.ai/code/session_011utN3x8yYUNDvkpGCEq5yD
Parts:
- C21, C25, C26, C27, C28, C29: footprint PicoGUS-THT:C_Disc_D5.0mm_W2.5mm_P5.00mm_0805_Hybrid -> Capacitor_THT:C_Disc_D5.0mm_W2.5mm_P5.00mm; Alternatives 0805 SMD (fits between the holes): Samsung CL21B104KBCNNNC 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 -> (none)
- C24: footprint PicoGUS-THT:C_Disc_D5.0mm_W2.5mm_P5.00mm_0805_Hybrid -> Capacitor_THT:C_Disc_D5.0mm_W2.5mm_P5.00mm; Alternatives 0805 SMD 25V X5R: Taiyo Yuden EMK212BJ106KG-T (DK 587-1295-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 -> (none)
- C30, C31: footprint PicoGUS-THT:C_Disc_D5.0mm_W2.5mm_P5.00mm_0805_Hybrid -> Capacitor_THT:C_Disc_D5.0mm_W2.5mm_P5.00mm; Alternatives THT: TDK FG28C0G1H101JNT06 (DK 445-173472-1-ND). 0805 SMD: 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 -> TDK FG28C0G1H101JNT06 (DK 445-173472-1-ND).
- R10, R11, R12, R13, R16, R19, R20, R9: footprint PicoGUS-THT:R_Axial_DIN0207_P10.16mm_0805_Hybrid -> Resistor_THT:R_Axial_DIN0207_L6.3mm_D2.5mm_P10.16mm_Horizontal; Alternatives 0805 SMD (fits between the holes): Yageo RC0805FR-0710KL (D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 -> (none)
- R14, R15: footprint PicoGUS-THT:R_Axial_DIN0207_P10.16mm_0805_Hybrid -> Resistor_THT:R_Axial_DIN0207_L6.3mm_D2.5mm_P10.16mm_Horizontal; Alternatives 0805 SMD (fits between the holes): Yageo RC0805FR-07100KL (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 -> (none)
- R21, R22: footprint PicoGUS-THT:R_Axial_DIN0207_P10.16mm_0805_Hybrid -> Resistor_THT:R_Axial_DIN0207_L6.3mm_D2.5mm_P10.16mm_Horizontal; Alternatives 0805 SMD (fits between the holes): Yageo RC0805FR-07100RL (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 -> (none)
- U10: footprint PicoGUS-THT:DIP-14_W7.62mm_TSSOP-14_Hybrid -> Package_DIP:DIP-14_W7.62mm; Alternatives DIP also as Rochester 2156-SN74AHCT126N-ND (58265). DigiKey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 -> Rochester 2156-SN74AHCT126N-ND (58265).; LCSC C155177 (SN74AHCT126PWR (TSSOP-14, fits inside the DIP)) -> C1548378
- U7: footprint PicoGUS-THT:DIP-14_W7.62mm_TSSOP-14_Hybrid -> Package_DIP:DIP-14_W7.62mm; Alternatives DIP also as Rochester 2156-SN74AHC00N-ND (21358). DigiKey T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 -> Rochester 2156-SN74AHC00N-ND (21358).; LCSC C7803 (SN74LVC00APWR (TSSOP-14, fits inside the DIP)) -> C2879122

Commit message: hw-tht: cleaner audio supplies, bipolar WT coupling caps, circuit-block groups
- DAC AVDD (U9 pin 8) gets its own rail behind ferrite bead FB3, with C13/C15
  at the pin; DVDD/CPVDD stay on the Pico 3V3.
- NE5532 +/-12 V from ISA through R23/R24 (10R) + C32/C33 (47uF) RC filters,
  C28/C29 0.1uF stay at the op-amp pins.
- C22/C23 WT coupling caps are now 10uF bipolar (Panasonic ECE-A1HN100U):
  the DC across them depends on the daughterboard.
- Every chip and its decoupling caps/resistors form a KiCad group.
- DAC pre-routes reworked (VNEG via B.Cu, XSMT via); RUN RC moved out of the
  Pico fan-in. Fully routed, 0 DRC errors, 0 unconnected.
- BOM: new lines for R23/R24, FB3, C32/C33; README has DigiKey cost in NOK.

Co-Authored-By: Claude Opus 5.5 <noreply@anthropic.com>
Claude-Session: https://claude.ai/code/session_011utN3x8yYUNDvkpGCEq5yD
Parts:
- removed C22, C23: 10uF, Capacitor_THT:CP_Radial_D5.0mm_P2.00mm, symbol Device:C_Polarized
- removed unit 5 of U10
- added C22, C23: 10uF bipolar, Capacitor_THT:C_Radial_D6.3mm_H11.0mm_P2.50mm, symbol Device:C
- added C32, C33: 47uF, Capacitor_THT:CP_Radial_D5.0mm_P2.00mm, symbol Device:C_Polarized
- added R23, R24: 10, Resistor_THT:R_Axial_DIN0207_L6.3mm_D2.5mm_P10.16mm_Horizontal, symbol Device:R
- added unit 3 of U10
Connections:
- net +12V: now also R23.1; no longer C28.1, U11.8 (V+)
- net +5V: now also U10.14 (VCC)
- net -12V: now also R24.1; no longer C29.2, U11.4 (V-)
- net GND: now also U10.7 (GND), C32.2, C33.1, U10.9; no longer U10.9
- net RESET: now also U10.10; no longer U10.10
- net WT_L: now also C22.1
- net WT_R: now also C23.1
- net ~{WT_RESET}: now also U10.8; no longer U10.8
- net at RV1.6: now also C23.2
- net at RV1.3: now also C22.2
- new net +12VA: C28.1, C32.1, R23.2, U11.8 (V+)
- new net -12VA: C29.2, C33.2, R24.2, U11.4 (V-)
Other:
- note added: "RV1 (dual 10k log) sets the WT level: pins 3/6 = CW end (signal), 1/4 = CCW end (GND). U11 sums PCM and WT at unity gain (inverting, 10k/10k) - no level loss, and the WT knob does not change the PCM level. C22/C23 (bipolar) block DC from the DB, R14/R15 keep them discharged when no DB is fitted. Output: 100R, DC-coupled like v1.2."
- note added: "U11 SUPPLY: ISA +/-12 V via R23/R24 (10R) + C32/C33 (47u), C28/C29 at the U11 pins"
- note removed: "RV1 (dual 10k log) sets the WT level: pins 3/6 = CW end (signal), 1/4 = CCW end (GND). U11 sums PCM and WT at unity gain (inverting, 10k/10k) - no level loss, and the WT knob does not change the PCM level. C22/C23 block DC from the DB, R14/R15 keep them discharged when no DB is fitted. Output: 100R, DC-coupled like v1.2."
- note removed: "U11 SUPPLY: ISA +/-12 V (place C28/C29 at U11)"
- moved on the sheet: U10E

Commit message: RV1: Bourns PTD902-2020K-A103 as primary part, Alps as alternative
Schematic fields (Manufacturer/MPN/DigiKey), BOM CSVs and DigiKey upload
files (1 and 10 boards) now use the Bourns pot (PTD902-2020K-A103-ND,
426 in stock, 24 kr vs 45 kr). Alps RK09712200HA and RK0971221Z0X are
listed as alternatives; the THT LCSC column keeps C470545 (Alps) since
LCSC does not carry the Bourns part. README cost tables updated.

Co-Authored-By: Claude Opus 5.5 <noreply@anthropic.com>
Claude-Session: https://claude.ai/code/session_011utN3x8yYUNDvkpGCEq5yD
Parts:
- RV1: DigiKey 4809-RK09712200HA-ND -> PTD902-2020K-A103-ND; MPN RK09712200HA -> PTD902-2020K-A103; Manufacturer Alps Alpine -> Bourns
Changed lines of the file:
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@@
 			)
 		)
-		(property "Manufacturer" "Alps Alpine"
+		(property "Manufacturer" "Bourns"
 			(at 152.4 104.14 0)
 			(hide yes)
@@
 			)
 		)
-		(property "MPN" "RK09712200HA"
+		(property "MPN" "PTD902-2020K-A103"
 			(at 152.4 104.14 0)
 			(hide yes)
@@
 			)
 		)
-		(property "DigiKey" "4809-RK09712200HA-ND"
+		(property "DigiKey" "PTD902-2020K-A103-ND"
 			(at 152.4 104.14 0)
 			(hide yes)
@@
 			)
 		)
-		(property "Manufacturer" "Alps Alpine"
+		(property "Manufacturer" "Bourns"
 			(at 152.4 139.7 0)
 			(hide yes)
@@
 			)
 		)
-		(property "MPN" "RK09712200HA"
+		(property "MPN" "PTD902-2020K-A103"
 			(at 152.4 139.7 0)
 			(hide yes)
@@
 			)
 		)
-		(property "DigiKey" "4809-RK09712200HA-ND"
+		(property "DigiKey" "PTD902-2020K-A103-ND"
 			(at 152.4 139.7 0)
 			(hide yes)
