File: hw-ne2k/PicoGUS-NE2K.kicad_sch (KiCad schematic)
At the start: 30 parts, among them J1 2x5 header, J3 Bus_ISA_8bit, J6 1x2 header, U1 Raspberry Pi Pico W, U10 74LVC2G06, U2 74LVC244, U3 SN74CB3T3257, U4 SN74CB3T3257, U5 74AHC14, U6 74LVC00, U7 74LVC1G00, U8 APS6404L-3SQR-SN

Commit message: hw-ne2k: placed (unrouted) board, BOM with DigiKey links, README, PDF
- PCB on the v1.2 outline: Pico W along the top with its antenna end
  toward the bracket (RF keep-out to the edge), USB-A (Molex 67643) at
  the bracket, boot ROM over the address fingers, bus logic over the data
  fingers. Routing in progress.
- J5 USB-A: Molex 0676432910 (DigiKey WM11258-ND); the PicoGUS 2.0 part is
  not sold by DigiKey and the Wurth part is out of stock.
- BOM-NE2K.csv + DigiKey upload files (1 and 10 boards), ~264 kr/board.
- Schematic PDF and README (Pico W/USB test points, antenna, boot ROM
  GPIO map and base/bank encoding, bracket changes).

Co-Authored-By: Claude Opus 5.5 <noreply@anthropic.com>
Claude-Session: https://claude.ai/code/session_011utN3x8yYUNDvkpGCEq5yD
Parts:
- J1: DigiKey TBD -> 10129381-910001BLF-ND
Changed lines of the file:
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@@
 			)
 		)
-		(property "DigiKey" "TBD"
+		(property "DigiKey" "10129381-910001BLF-ND"
 			(at 167.64 78.105 0)
 			(hide yes)
