File: hw-ne2k/bootrom.kicad_sch (KiCad schematic)
At the start: 16 parts, among them J2 1x2 header, J5 USB-A, U13 SST39SF010A, U14 74HCT688, U15 74AHCT245, U16 74AHCT1G08, U17 USBLC6-2SC6

Commit message: hw-ne2k: placed (unrouted) board, BOM with DigiKey links, README, PDF
- PCB on the v1.2 outline: Pico W along the top with its antenna end
  toward the bracket (RF keep-out to the edge), USB-A (Molex 67643) at
  the bracket, boot ROM over the address fingers, bus logic over the data
  fingers. Routing in progress.
- J5 USB-A: Molex 0676432910 (DigiKey WM11258-ND); the PicoGUS 2.0 part is
  not sold by DigiKey and the Wurth part is out of stock.
- BOM-NE2K.csv + DigiKey upload files (1 and 10 boards), ~264 kr/board.
- Schematic PDF and README (Pico W/USB test points, antenna, boot ROM
  GPIO map and base/bank encoding, bracket changes).

Co-Authored-By: Claude Opus 5.5 <noreply@anthropic.com>
Claude-Session: https://claude.ai/code/session_011utN3x8yYUNDvkpGCEq5yD
Parts:
- J5: footprint Connector_USB:USB_A_Wuerth_614004134726_Horizontal -> Connector_USB:USB_A_Molex_67643_Horizontal; Alternatives (none) -> Wurth 614004134726 (DK 732-2731-ND, different footprint).; DigiKey TBD -> WM11258-ND; MPN 614004134726 -> 0676432910; Manufacturer Wurth Elektronik -> Molex
- U14: DigiKey TBD -> 296-24357-1-ND
- U15: DigiKey TBD -> 296-1118-1-ND
- U16: DigiKey TBD -> 296-1113-1-ND
- U17: DigiKey TBD -> 497-5235-1-ND
Changed lines of the file:
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@@
 			)
 		)
-		(property "DigiKey" "TBD"
+		(property "DigiKey" "296-1113-1-ND"
 			(at 50.8 58.42 0)
 			(hide yes)
@@
 			)
 		)
-		(property "DigiKey" "TBD"
+		(property "DigiKey" "296-24357-1-ND"
 			(at 50.8 110.49 0)
 			(hide yes)
@@
 			)
 		)
-		(property "DigiKey" "TBD"
+		(property "DigiKey" "296-1118-1-ND"
 			(at 200.66 101.6 0)
 			(hide yes)
@@
 			)
 		)
-		(property "Footprint" "Connector_USB:USB_A_Wuerth_614004134726_Horizontal"
+		(property "Footprint" "Connector_USB:USB_A_Molex_67643_Horizontal"
 			(at 228.6 134.62 0)
 			(hide yes)
@@
 			)
 		)
-		(property "Manufacturer" "Wurth Elektronik"
+		(property "Manufacturer" "Molex"
 			(at 228.6 134.62 0)
 			(hide yes)
@@
 			)
 		)
-		(property "MPN" "614004134726"
+		(property "MPN" "0676432910"
 			(at 228.6 134.62 0)
 			(hide yes)
@@
 			)
 		)
-		(property "DigiKey" "TBD"
+		(property "DigiKey" "WM11258-ND"
+			(at 228.6 134.62 0)
+			(hide yes)
+			(show_name no)
+			(do_not_autoplace no)
+			(effects
+				(font
+					(size 1.27 1.27)
+				)
+			)
+		)
+		(property "Alternatives" "Wurth 614004134726 (DK 732-2731-ND, different footprint)."
 			(at 228.6 134.62 0)
 			(hide yes)
@@
 			)
 		)
-		(property "DigiKey" "TBD"
+		(property "DigiKey" "497-5235-1-ND"
 			(at 266.7 139.7 0)
 			(hide yes)
