File: hw-tht-v1.3.1/wavetable.kicad_sch (KiCad schematic)
At the start: 33 parts, among them J8 SJ1-3535NG-GR, J9 Waveblaster, U10 74AHCT126, U11 NE5532, U7 74AHC00

Commit message: THT rev B: user's new placement; USB port and Waveblaster standoff holes dropped
- PicoGUS-THT.kicad_pcb: the user's rev B placement (Pico moved down, bracket
  parts and mixer regrouped), unrouted
- USB host port removed again (usb.kicad_sch, J11, F1, C34, C35, U12); U1 back
  on the v1.3.0 Pico symbol and RPi_Pico_SMD_TH footprint
- J9 on the new Wavetable_NoMountingHoles footprint (no daughterboard standoff
  holes; the far one landed in U4); standoff and screws dropped from the BOM
- card outline: the 6.35 mm Edge.Cuts step at x 197.41 next to the ISA
  fingers had been dragged off the board in the upload; restored
- design rules identical to v1.3.0
- BOM, DigiKey uploads, socket BOM, schematic PDF and README updated

Co-Authored-By: Claude Opus 5.5 <noreply@anthropic.com>
Claude-Session: https://claude.ai/code/session_011utN3x8yYUNDvkpGCEq5yD
Parts:
- J9: footprint PiGUS library:Wavetable -> PiGUS library:Wavetable_NoMountingHoles
Changed lines of the file:
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@@
 			)
 		)
-		(property "Footprint" "PiGUS library:Wavetable"
+		(property "Footprint" "PiGUS library:Wavetable_NoMountingHoles"
 			(at 60.96 90.17 0)
 			(hide yes)
