File: hw-tht-v1.3.1/audio.kicad_sch (KiCad schematic)
At the start: 14 parts, among them J10 GY-PCM5102, U9 PCM5100A

Commit message: THT rev B: U9 CPVDD cap, U12 flow-through at J11, wide GND strap for finger B10
- C36 (new, 0.1 uF X7R 0603, Yageo CC0603KRX7R9BB104 / LCSC C14663 basic part) right under U9 pins 1-3:
  CPVDD -> C36 -> CPGND loop ~6.6 mm (before: nearest +3V3 cap C4 23.6 mm of track away). C16 0.5 mm left,
  R7 0.4 mm down, CPGND via below C36, two GND stitching vias for the front pour west of U9. Schematic
  (audio sheet), BOM and DigiKey uploads updated; CPVDD stays on +3V3 as on v1.2/v1.3.0.
- U12 (USBLC6-2SC6) moved right behind J11 and wired flow-through (no stubs; was 13/26 mm), GND via at
  pin 2, VBUS via to J11.1; C35 below U12, C34 0.2 mm up; USB pair re-routed and re-locked (42.2/42.5 mm,
  matched to 0.28 mm); ~RIOR, ~SPI_CS, SPI_RX re-routed locally; board-level pin-1 dot for U12.
- GND finger B10: 1.5-3 mm B.Cu strap into the U3/U4 pour (link 12.6 -> 3.5 mOhm; B10 to U3/U4 GND
  21/18 -> 11/8 mOhm).
- README: the three changes, U12/C36 assembly notes.

DRC with schematic parity: 0 errors, 0 unconnected; ERC 0 errors. No audio net has another net within 0.5 mm.

Co-Authored-By: Claude Opus 5.5 <noreply@anthropic.com>
Claude-Session: https://claude.ai/code/session_011utN3x8yYUNDvkpGCEq5yD
Parts:
- added C36: 0.1uF, Capacitor_SMD:C_0603_1608Metric, symbol Device:C_Small
Connections:
- net +3V3: now also C36.1
- net GND: now also C36.2
Other:
- note added: "C36: CPVDD (U9 pin 1) decoupling, right at pins 1 (CPVDD) and 3 (CPGND)"
- note added: "OPTION: GY-PCM5102 module (J10) INSTEAD OF the on-board DAC. Fit EITHER U9 + C12-C20 + C36 + FB3 + R7/R8 OR the module - never both (two DAC outputs would fight). The module has its own 470R/2.2nF output filter. Module solder jumpers: H1=L H2=L H3=H H4=L."
- note removed: "OPTION: GY-PCM5102 module (J10) INSTEAD OF the on-board DAC. Fit EITHER U9 + C12-C20 + FB3 + R7/R8 OR the module - never both (two DAC outputs would fight). The module has its own 470R/2.2nF output filter. Module solder jumpers: H1=L H2=L H3=H H4=L."
