File: hw-tht-v1.3.2/PicoGUS-THT.kicad_sch (KiCad schematic)
At the start: 38 parts, among them J1 IRQDMA_JP, J3 Bus_ISA_8bit, J5 SJ1-3535NG, J6 UART_TX, J7 USB power jumper, U1 Pico, U10 74AHCT126, U2 74AHC244, U3 SN74CB3T3257, U4 SN74CB3T3257, U5 74AHC14, U6 74AHC00, U7 74AHC00, U8 APS6404L-3SQR-SN

Commit message: THT v1.3.2: adopt the 102 mm placement (unrouted) with 3D models
The board now holds the new hand placement on a 102.0 mm outline in place
of the routed 103.7 mm layout (that one stays in 8dbb6c6). It has no
tracks or vias yet and has to be routed again.

- Logic column in line with U2 with the decoupling discs between the
  chips, R18/R5/R6/R17 vertical, DAC group 15 mm left, FB3 vertical,
  copper logo along the top edge over LINE OUT, several labels moved.
- C8/C10 back to the v1.3.1 Murata through-hole discs, in a row above
  U8 (schematic fields, BOM and DigiKey upload files updated).
- Back princess artwork removed (to be UV printed); back texts kept.
- Bracket end trimmed 1.84 mm (JLCPCB prices <= 102 mm lower). H1/H2
  1.70 mm, J8 1.10, J5 0.90, Pico 1.35 (with its slots and rule areas),
  U4 0.45 and U3 0.35 mm moved so copper stays >= 0.35 mm from the edge.
  The bracket tab holes are now 7.03 mm behind the plate: it needs a
  bracket with longer tabs (3D-printed).
- U1 uses the new RPi_Pico_SMD_TH_USB_NoSWD footprint (no SMD pads for
  the unconnected SWD castellations, tighter courtyard).
- 3D models for every part: CUI jacks (J5 a black copy of the CUI
  model), Alps RK09712 pot, a generated MF-R050 model, U3/U4/U9 socket +
  adapter stacks exported from the adapter PCBs, KiCad's Pico model,
  J9's model path fixed. Library footprints carry the same models.
- Schematic title note and PDF updated; README rewritten for the
  adopted, unrouted layout.

DRC with schematic parity: 12 accepted courtyard overlaps in the logic
column, 309 unconnected (unrouted), warnings only otherwise; ERC as before.

Co-Authored-By: Claude Opus 5.5 <noreply@anthropic.com>
Claude-Session: https://claude.ai/code/session_011utN3x8yYUNDvkpGCEq5yD
Parts:
- C10: footprint Capacitor_SMD:C_0805_2012Metric -> Capacitor_THT:C_Disc_D5.0mm_W2.5mm_P5.00mm; Alternatives DigiKey line is KYOCERA AVX 08055C105KAT2A (same 1uF 50V X7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 -> (none); DigiKey 478-KGM21AR71H105KUCT-ND -> 490-9146-1-ND; LCSC C28323 -> C1620132; MPN CL21B105KBFNNNE -> RDER71H105K2M1H03A; Manufacturer Samsung Electro-Mechanics -> Murata
- C8: footprint Capacitor_SMD:C_0805_2012Metric -> Capacitor_THT:C_Disc_D5.0mm_W2.5mm_P5.00mm; DigiKey 311-1140-1-ND -> 490-9144-1-ND; LCSC C49678 -> C527620; MPN CC0805KRX7R9BB104 -> RDER71H104K0M1H03A; Manufacturer Yageo -> Murata
- U1: footprint PiGUS library:RPi_Pico_SMD_TH_USB -> PiGUS library:RPi_Pico_SMD_TH_USB_NoSWD
Changed lines of the file:
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@@
 	(title_block
 		(title "PicoGUS THT")
-		(date "2026-10-23")
+		(date "2026-10-28")
 		(rev "v1.3.2")
 		(comment 1 "Through-hole variant of PicoGUS v1.2 with Waveblaster header and USB host port")
-		(comment 2 "U3/U4/U9 on 300-mil DIP adapters; SMD: U8, C8/C10 0805 (back), U12 opt.")
+		(comment 2 "U3/U4/U9 on 300-mil DIP adapters; SMD: U8, U12 opt.")
 	)
 	(text "Saves PIO instructions due to JMP limitations"
@@
 			)
 		)
-		(property "Footprint" "Capacitor_SMD:C_0805_2012Metric"
+		(property "Footprint" "Capacitor_THT:C_Disc_D5.0mm_W2.5mm_P5.00mm"
 			(at 63.8302 190.5 0)
 			(hide yes)
@@
 			)
 		)
-		(property "Description" "1uF 50V X7R 0805 MLCC: U8/+3V3 bulk, on the BACK under U8"
+		(property "Description" "1uF 50V X7R radial MLCC, 5.0 mm pitch: U8/+3V3 bulk, above U8"
 			(at 62.865 186.69 0)
 			(hide yes)
@@
 			)
 		)
-		(property "Manufacturer" "Samsung Electro-Mechanics"
+		(property "Manufacturer" "Murata"
 			(at 62.865 186.69 0)
 			(hide yes)
@@
 			)
 		)
-		(property "MPN" "CL21B105KBFNNNE"
+		(property "MPN" "RDER71H105K2M1H03A"
 			(at 62.865 186.69 0)
 			(hide yes)
@@
 			)
 		)
-		(property "DigiKey" "478-KGM21AR71H105KUCT-ND"
+		(property "DigiKey" "490-9146-1-ND"
 			(at 62.865 186.69 0)
 			(hide yes)
@@
 			)
 		)
-		(property "LCSC" "C28323"
+		(property "LCSC" "C1620132"
 			(at 62.865 186.69 0)
 			(hide yes)
@@
 			)
 		)
-		(property "Alternatives" "DigiKey line is KYOCERA AVX 08055C105KAT2A (same 1uF 50V X7R 0805): Samsung CL21B105KBFNNNE (DigiKey 1276-1029-1-ND) had no DigiKey stock on 2026-10-23. LCSC C28323 is a JLCPCB basic part."
-			(at 62.865 186.69 0)
-			(hide yes)
-			(show_name no)
-			(do_not_autoplace no)
-			(effects
-				(font
-					(size 1.27 1.27)
-				)
-			)
-		)
 		(pin "1"
 		)
@@
 			)
 		)
-		(property "Footprint" "Capacitor_SMD:C_0805_2012Metric"
+		(property "Footprint" "Capacitor_THT:C_Disc_D5.0mm_W2.5mm_P5.00mm"
 			(at 53.6702 190.5 0)
 			(hide yes)
@@
 			)
 		)
-		(property "Description" "0.1uF 50V X7R 0805 MLCC: U8 decoupling, on the BACK under U8"
+		(property "Description" "0.1uF 50V X7R radial MLCC, 5.0 mm pitch: U8 decoupling, above U8"
 			(at 52.705 186.69 0)
 			(hide yes)
@@
 			)
 		)
-		(property "Manufacturer" "Yageo"
+		(property "Manufacturer" "Murata"
 			(at 52.705 186.69 0)
 			(hide yes)
@@
 			)
 		)
-		(property "MPN" "CC0805KRX7R9BB104"
+		(property "MPN" "RDER71H104K0M1H03A"
 			(at 52.705 186.69 0)
 			(hide yes)
@@
 			)
 		)
-		(property "DigiKey" "311-1140-1-ND"
+		(property "DigiKey" "490-9144-1-ND"
 			(at 52.705 186.69 0)
 			(hide yes)
@@
 			)
 		)
-		(property "LCSC" "C49678"
+		(property "LCSC" "C527620"
 			(at 52.705 186.69 0)
 			(hide yes)
@@
 			)
 		)
-		(property "Footprint" "PiGUS library:RPi_Pico_SMD_TH_USB"
+		(property "Footprint" "PiGUS library:RPi_Pico_SMD_TH_USB_NoSWD"
 			(at 109.22 61.595 90)
 			(hide yes)
