File: hw-tht-v2.1/PicoGUS-THT.kicad_pcb (KiCad board)
At the start: 2 copper layers, 102.9 x 96.7 mm, 90 parts, among them J1 Bus_ISA_8bit, J10 RUN, J2 SWD, J3 IRQ/DMA, J4 UART_TX, J5 USB-A host, J6 USB-C program, J7 SJ1-3535NG, J8 Waveblaster, J9 SJ1-3535NG-GR, SW1 BOOTSEL, U1 SN74CB3T3257, U10 PCM5100A, U11 NE5532, U12 Core2350B, U13 M62429L, U2 SN74CB3T3257, U3 74AHC14, U4 74AHC00, U5 74AHC00, U6 74AHCT126, U7 74AHC244, U9 MCP1826S-3302E/AB

Commit message: THT v2.1: routed 4-layer board with AGND/AVDD islands, silkscreen
- Routed on 4 layers (In1 GND, In2 +3V3, as v2.0): Freerouting for most
  nets, the rest with stricter rules: nothing between the ISA gold
  fingers, vias above the finger tops, digital tracks kept out of the
  audio section. A few short bus hops use In2 (now layer type "mixed").
- AGND island on In1 and AVDD island on In2 under the audio section,
  joined to GND/+3V3 only at FB3/FB4, as v2.0. I2S, MIDI and the
  Waveblaster reset re-routed to cross the islands as little as
  possible. GND finger vias into the plane; the Waveblaster's digital
  GND pocket tied to the main plane.
- Silkscreen: PicoGUS v2.1 THT title, LINE OUT label, back block with
  copyright, licence, URL and thanks.
- DRC with schematic parity: 0 errors, 0 unconnected, 0 parity issues
  (36 warnings for connector silkscreen past the bracket edge).
- jlcpcb.sh: export the inner copper layers of multilayer boards.
- README: status, planes, layout status; front and back renders.

Co-Authored-By: Claude Opus 5.5 <noreply@anthropic.com>
Claude-Session: https://claude.ai/code/session_013W5uqvghZgJXEB5tgmrp98
Routing:
- net +5V: track 0.00 -> 270.2 mm, vias 0 -> 3
- net AGND: track 0.00 -> 253.7 mm, vias 0 -> 2
- net UART_TX: track 0.00 -> 145.2 mm, vias 0 -> 2
- net -12V: track 0.00 -> 141.0 mm
- net +12V: track 0.00 -> 129.6 mm, vias 0 -> 1
- net DACK: track 0.00 -> 123.7 mm, vias 0 -> 3
- net RESET: track 0.00 -> 100.0 mm, vias 0 -> 5
- net AVDD: track 0.00 -> 98.4 mm
- net ADS: track 0.00 -> 95.3 mm, vias 0 -> 3
- net RUN: track 0.00 -> 86.3 mm, vias 0 -> 1
- net BCK: track 0.00 -> 79.4 mm, vias 0 -> 6
- net /VBUS_PRG: track 0.00 -> 78.3 mm, vias 0 -> 1
- net ~{RIOW}: track 0.00 -> 76.9 mm, vias 0 -> 3
- net RI/OCHRDY: track 0.00 -> 76.6 mm, vias 0 -> 1
- net ~{RIOR}: track 0.00 -> 76.1 mm
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- added copper zone on In2.Cu, net +3V3
- added copper zone on In1.Cu, net AGND
- added copper zone on In2.Cu, net AVDD
- added copper zone on In1.Cu, net GND
Other:
- copper layers 2 -> 4
- board text added: "LINE OUT"
- board text added: "Licensed under CERN-OHL-P v2"
- board text added: "PicoGUS"
- board text added: "PicoGUS v2.1 THT"
- board text added: "Thanks to polpo and all"
- board text added: "Vidar Waagbø (waagbo)"
- board text added: "github.com/polpo/picogus"
- board text added: "the PicoGUS contributors."
- board text added: "v2.1 THT"
- board text added: "© 2023-2026 Ian Scott (polpo),"
- board text removed: "v2.1"
