File: hw-tht-v1.3.2/adapters/TSSOP20-DIP20-300mil/TSSOP20-DIP20-300mil.kicad_pcb (KiCad board)
At the start: 2 copper layers, 10.2 x 25.4 mm, 8 parts, among them J1 DIP-20 pins (10+10, 300 mil), U1 PCM5100A

Commit message: THT v1.3.2 adapters: generic silkscreen
Drop the reference designators (U3/U4, U9) and the version number from
both adapter boards. The bottom now says what each board does, centred
on two lines (TSSOP-16 / DIP-16, TSSOP-20 / DIP-20), and still names the
chip it carries on PicoGUS. Copper unchanged; DRC with schematic parity
clean. Assembly views, DRC reports and the adapter STEP models (with
silkscreen) regenerated; README updated.

Co-Authored-By: Claude Opus 5.5 <noreply@anthropic.com>
Claude-Session: https://claude.ai/code/session_011utN3x8yYUNDvkpGCEq5yD
Other:
- board text added: "PCM5100A"
- board text added: "TSSOP-20 DIP-20"
- board text removed: "PCM5100A TSSOP20"
- board text removed: "PicoGUS v1.3.2 U9"
- board text removed: "U9"
Changed lines of the file:
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@@
 				(font
 					(size 1.27 1.27)
+					(thickness 0.15)
 				)
 			)
@@
 				(font
 					(size 1.27 1.27)
+					(thickness 0.15)
 				)
 			)
@@
 				(font
 					(size 1.27 1.27)
+					(thickness 0.15)
 				)
 			)
@@
 				(font
 					(size 1.27 1.27)
+					(thickness 0.15)
 				)
 			)
@@
 				(font
 					(size 1.27 1.27)
+					(thickness 0.15)
 				)
 			)
@@
 				(font
 					(size 1.27 1.27)
+					(thickness 0.15)
 				)
 			)
@@
 				(font
 					(size 1.27 1.27)
+					(thickness 0.15)
 				)
 			)
@@
 				(font
 					(size 1.27 1.27)
+					(thickness 0.15)
 				)
 			)
@@
 				(font
 					(size 1.27 1.27)
+					(thickness 0.15)
 				)
 			)
@@
 				(font
 					(size 1.27 1.27)
+					(thickness 0.15)
 				)
 			)
@@
 				(font
 					(size 1.27 1.27)
+					(thickness 0.15)
 				)
 			)
@@
 				(font
 					(size 1.27 1.27)
+					(thickness 0.15)
 				)
 			)
@@
 				(font
 					(size 1.27 1.27)
+					(thickness 0.15)
 				)
 			)
@@
 				(font
 					(size 1.27 1.27)
+					(thickness 0.15)
 				)
 			)
@@
 				(font
 					(size 1.27 1.27)
+					(thickness 0.15)
 				)
 			)
@@
 				(font
 					(size 1.27 1.27)
+					(thickness 0.15)
 				)
 			)
@@
 				(font
 					(size 1.27 1.27)
+					(thickness 0.15)
 				)
 			)
@@
 				(font
 					(size 1.27 1.27)
+					(thickness 0.15)
 				)
 			)
@@
 				(font
 					(size 1.27 1.27)
+					(thickness 0.15)
 				)
 			)
@@
 				(font
 					(size 1.27 1.27)
+					(thickness 0.15)
 				)
 			)
@@
 				(font
 					(size 1.27 1.27)
+					(thickness 0.15)
 				)
 			)
@@
 				(font
 					(size 1.27 1.27)
+					(thickness 0.15)
 				)
 			)
@@
 				(font
 					(size 1.27 1.27)
+					(thickness 0.15)
 				)
 			)
@@
 				(font
 					(size 1.27 1.27)
+					(thickness 0.15)
 				)
 			)
@@
 				(font
 					(size 1.27 1.27)
+					(thickness 0.15)
 				)
 			)
@@
 				(font
 					(size 1.27 1.27)
+					(thickness 0.15)
 				)
 			)
@@
 				(font
 					(size 1.27 1.27)
+					(thickness 0.15)
 				)
 			)
@@
 		)
 	)
-	(gr_text "U9"
-		(at 103.61 100 0)
-		(layer "F.SilkS")
-		(effects
-			(font
-				(size 1 0.9)
-				(thickness 0.15)
-			)
-		)
-	)
-	(gr_text "PicoGUS v1.3.2  U9"
-		(at 101.76 115.63 90)
+	(gr_text "TSSOP-20\nDIP-20"
+		(at 103.81 102.93 0)
 		(layer "B.SilkS")
 		(effects
 			(font
-				(size 1 0.75)
+				(size 1 0.7)
 				(thickness 0.15)
 			)
@@
 		)
 	)
-	(gr_text "PCM5100A  TSSOP20"
-		(at 105.86 111.83 90)
+	(gr_text "PCM5100A"
+		(at 105.86 111.43 90)
 		(layer "B.SilkS")
 		(effects
